Commit message: ball_chaser added

File: my_robot/urdf/my_robot.xacro (robot description, xacro)
@@ -1,4 +1,4 @@
 <?xml version='1.0'?>
-<robot name="my_robot" xmlns:xacro="http://www.ros.org/wiki/xacro">
+  <robot name="my_robot" xmlns:xacro="http://www.ros.org/wiki/xacro">
   <xacro:include filename="$(find my_robot)/urdf/my_robot.gazebo" />
   <link name="robot_footprint"></link>
@@ -9,5 +9,5 @@
   </joint>
   <joint name="camera_joint" type="fixed">
-    <origin xyz="0.2 0 0" rpy="0 0 0"/>
+    <origin xyz="0.21 0 0" rpy="0 0 0"/>
     <axis xyz="0 1 0" rpy="0 0 0"/>
     <parent link="chassis"/>
@@ -147,5 +147,5 @@
         <origin xyz="0 0 0" rpy="0 0 0"/>
         <geometry>
-          <box size=".05 .05 .05"/>
+          <box size=".01 .14 .01"/>
         </geometry>
       </collision>
@@ -154,5 +154,5 @@
         <geometry>
           <mesh filename="package://my_robot/meshes/realsense.dae"/>
-          <box size=".05 .05 .05"/>
+          <box size=".01 .14 .01"/>
         </geometry>
       </visual>
@@ -184,12 +184,3 @@
       </visual>
     </link>
-    <gazebo reference="left_wheel">
-      <material>Gazebo/Orange</material>
-    </gazebo>
-    <gazebo reference="right_wheel">
-      <material>Gazebo/Orange</material>
-    </gazebo>
-    <gazebo reference="chassis">
-      <material>Gazebo/Orange</material>
-    </gazebo>
 </robot>
